Commit message: misc fixes

File: tetra/gello-left.urdf (robot description, URDF)
Before this commit: robot onshape, 8 links, 7 joints
Links:
- removed link gopromount_l
- added link manus_glove_mount, mass 0
- link 1l: geometry 
- link 2l: mass 0.01926664587663814987 -> 0.043917844969380323561; geometry 
- link 3l: geometry 
- link 4l: geometry 
- link 5l: geometry 
- link 6l: geometry 
Joints:
- joint 1: limit effort=1 velocity=20 -> lower=-6.28318530718 upper=6.28318530718 effort=1 velocity=20; origin xyz=0.032794658465675544101 0.0073076307334959261786 0.11016039202600289015 rpy=3.1415926535897926719 4.1343810392342985243e-16 -1.570796326794896336 -> xyz=0.032794658465675544101 0.0073076307334959261786 0.11016039202600289015 rpy=3.1415926535897926719 4.1343810392342935939e-16 -1.570796326794896336
- joint 2: limit effort=1 velocity=20 -> lower=-6.28318530718 upper=6.28318530718 effort=1 velocity=20; origin xyz=-3.4694469519536141888e-17 0.022674999999999896627 -0.056199999999999999956 rpy=-1.57079632679489678 -2.4599427120222544936e-16 -3.1415926535897917837 -> xyz=-5.2041704279304212832e-17 0.022674999999999789074 -0.056199999999999999956 rpy=-1.57079632679489678 -2.4599427120222495632e-16 -3.1415926535897917837
- joint 3: limit effort=1 velocity=20 -> lower=-6.28318530718 upper=6.28318530718 effort=1 velocity=20; origin xyz=-0.023350000000000079026 0.27644999999999997353 -0.010499999999999896569 rpy=4.9303806576313259734e-32 2.2524931719504640392e-31 0 -> xyz=-0.023350000000000096373 0.27644999999999997353 -0.010500000000000004122 rpy=4.9303806576313259734e-32 2.2524931719504640392e-31 0
- joint 4: limit effort=1 velocity=20 -> lower=-6.28318530718 upper=6.28318530718 effort=1 velocity=20
- joint 5: limit effort=1 velocity=20 -> lower=-6.28318530718 upper=6.28318530718 effort=1 velocity=20
- joint 6: child gopromount_l -> manus_glove_mount; limit effort=1 velocity=20 -> lower=-6.28318530718 upper=6.28318530718 effort=1 velocity=20; origin xyz=-0.031650000000000066969 -0.065150000000000041211 0.054825000000000054245 rpy=1.570796326794896558 1.5866786711865396986e-17 3.141592653589793116 -> xyz=-0.031649999999999844924 -0.065150000000000041211 0.024999999999999997918 rpy=1.57079632679489678 -1.1250275051041753606e-16 3.1415926535897926719
- joint base_fixed: origin (none) -> xyz=0 0 0 rpy=0 0 0

File: tetra/gello-right.urdf (robot description, URDF)
Before this commit: robot onshape, 8 links, 7 joints
Links:
- removed link part_14
- added link manus_glove_mount, mass 0
- link 1r: geometry 
- link 2r: mass 0.019266645876638163748 -> 0.043917844969380316622; geometry 
- link 3r: geometry 
- link 4r: geometry 
- link 5r: geometry 
- link 6r: geometry 
Joints:
- joint 1: limit effort=1 velocity=20 -> lower=-6.28318530718 upper=6.28318530718 effort=1 velocity=20; origin xyz=-0.0076800387769155311832 0.10344814280253467054 0.021712491098799052702 rpy=3.141592653589793116 2.618469836202695248e-17 -1.5707963267948958919 -> xyz=-0.0076800387769155329179 0.10344814280253465666 0.021712491098799056172 rpy=3.141592653589793116 4.8572882273213452035e-17 -1.4359026091043931572
- joint 2: limit effort=1 velocity=20 -> lower=-6.28318530718 upper=6.28318530718 effort=1 velocity=20; origin xyz=-1.3877787807814456755e-17 0.022674999999999955608 -0.056200000000000013833 rpy=1.570796326794896558 3.4694469519530872544e-17 -1.1301130136656770669e-16 -> xyz=-1.1102230246251565404e-16 0.02267499999999993826 -0.056200000000000013833 rpy=1.570796326794896558 2.775620056149426907e-17 -3.6082248300317774918e-16
- joint 3: limit effort=1 velocity=20 -> lower=-6.28318530718 upper=6.28318530718 effort=1 velocity=20; origin xyz=-0.023349999999999995759 -0.27644999999999991802 -0.010499999999999926059 rpy=-2.4651903288156684605e-32 -9.7175910280077043601e-32 9.3985381286097361425e-32 -> xyz=-0.023349999999999981881 -0.27644999999999991802 -0.010500000000000241779 rpy=-3.4497645201609948565e-20 8.3561638130300710792e-17 -0.0018071395069734338609
- joint 4: limit effort=1 velocity=20 -> lower=-6.28318530718 upper=6.28318530718 effort=1 velocity=20; origin xyz=-0.2491500000000000381 -5.5511151231257827021e-17 0.021587499999999908845 rpy=3.141592653589793116 -1.570796326794896558 0 -> xyz=-0.24915000000000014913 1.6653345369377348106e-16 0.021587499999999960887 rpy=-3.141592653589793116 -1.570796326794896336 0
- joint 5: limit effort=1 velocity=20 -> lower=-6.28318530718 upper=6.28318530718 effort=1 velocity=20; origin xyz=-0.054425000000000001155 1.1102230246251565404e-16 -0.050500000000000044853 rpy=-3.141592653589793116 -1.570796326794896558 0 -> xyz=-0.054425000000000001155 0 -0.050500000000000155875 rpy=-1.5707963267949109909 -1.5572544369178140666 -1.5707963267948739094
- joint 6: child part_14 -> manus_glove_mount; limit effort=1 velocity=20 -> lower=-6.28318530718 upper=6.28318530718 effort=1 velocity=20; origin xyz=-0.031650000000000011458 0.065150000000000041211 0.054825000000000040368 rpy=1.570796326794896558 -8.8297424927219175422e-16 -1.8180778675015539296e-31 -> xyz=-0.031650000000000788614 0.065149999999999763656 0.02500000000000011241 rpy=1.570796326794896336 5.4442909851799711031e-16 5.0827397846120378841e-16
- joint base_fixed: origin (none) -> xyz=0 0 0 rpy=0 0 0
